Commit message: robot localization

File: robot-localization/urdf/camera_front.urdf.xacro (robot description, xacro)
@@ -1,6 +1,58 @@
-<xacro name="camera">
-    <link name="">
+<?xml version="1.0"?>
+<robot xmlns:xacro="https://www.ros.org/wiki/xacro" name="rover">
+<xacro:macro name="front_camera" params="name parent">
+    <link name="${name}_link">
+        <visual>
+            <geometry>
+                <box size="0.05 0.05 0.05" />
+            </geometry>
+            <material>
+                <color rgba="0.3 0.3 0.3 1" />
+            </material>
+        </visual>
+        <inertial>
+            <mass value="0.01" />
+            <inertia ixx="0.0001" ixy="0.0" ixz="0.0"
+                     iyy="0.0001" iyz="0.0" izz="0.0001" />
+        </inertial>
     </link>
-    <joint name="">
+    <joint name="${name}_joint" type="fixed">
+        <parent link="${parent}"/>
+        <child link="${name}_link"/>
+        <origin xyz="0.1 0 0.2" rpy="0 0 0"/>
     </joint>
-</xacro>
+    <gazebo reference="${name}_link">
+        <sensor type="camera" name="front_camera">
+            <always_on>true</always_on>
+            <update_rate>30</update_rate>
+            <visualize>true</visualize>
+            <camera>
+                <horizontal_fov>1.3962634</horizontal_fov>
+                <image>
+                    <width>640</width>
+                    <height>480</height>
+                    <format>R8G8B8</format>
+                </image>
+                <clip>
+                    <near>0.02</near>
+                    <far>50</far>
+                </clip>
+            </camera>
+            <plugin name="${name}_controller" filename="libgazebo_ros_camera.so">
+                <ros>
+                    <namespace>/</namespace>
+                    <argument>camera</argument>
+                </ros>
+                <camera_name>front_camera</camera_name>
+                <frame_name>camera_link</frame_name>
+                <hack_baseline>0.0</hack_baseline>
+                <distortion_k1>0.0</distortion_k1>
+                <distortion_k2>0.0</distortion_k2>
+                <distortion_k3>0.0</distortion_k3>
+                <distortion_t1>0.0</distortion_t1>
+                <distortion_t2>0.0</distortion_t2>
+            </plugin>
+        </sensor>
+    </gazebo>
+</xacro:macro>
+</robot>

File: robot-localization/urdf/wheel_front_left.urdf.xacro (robot description, xacro)
@@ -10,4 +10,5 @@
                 <color rgba="0.0 1.0 0.0 1" />
             </material>
+            <origin rpy="1.5708 0 0" />
         </visual>
         <collision>
@@ -24,5 +25,5 @@
         <parent link="${parent}"/>
         <child link="${name}_wheel"/>
-        <origin xyz="0.25 0.2 0" />
+        <origin xyz="0.75 0.4 0" />
         <axis xyz="0 1 0"/>
     </joint>

File: robot-localization/urdf/wheel_front_right.urdf.xacro (robot description, xacro)
@@ -10,4 +10,5 @@
                 <color rgba="0.0 1.0 0.0 1" />
             </material>
+            <origin rpy="1.5708 0 0" />
         </visual>
         <collision>
@@ -24,5 +25,5 @@
         <parent link="${parent}"/>
         <child link="${name}_wheel"/>
-        <origin xyz="0.25 0.2 0" />
+        <origin xyz="0.75 -0.4 0" />
         <axis xyz="0 1 0"/>
     </joint>

File: robot-localization/urdf/wheel_rear_left.urdf.xacro (robot description, xacro)
@@ -10,4 +10,5 @@
                 <color rgba="0.0 1.0 0.0 1" />
             </material>
+            <origin rpy="1.5708 0 0" />
         </visual>
         <collision>
@@ -24,5 +25,5 @@
         <parent link="${parent}"/>
         <child link="${name}_wheel"/>
-        <origin xyz="0.25 0.2 0"/>
+        <origin xyz="-0.75 0.4 0"/>
         <axis xyz="0 1 0"/>
     </joint>

File: robot-localization/urdf/wheel_rear_right.urdf.xacro (robot description, xacro)
@@ -10,4 +10,5 @@
                 <color rgba="0.0 1.0 0.0 1" />
             </material>
+            <origin rpy="1.5708 0 0" />
         </visual>
         <collision>
@@ -24,5 +25,5 @@
         <parent link="${parent}"/>
         <child link="${name}_wheel"/>
-        <origin xyz="0.25 0.2 0" />
+        <origin xyz="-0.75 -0.4 0" />
         <axis xyz="0 1 0"/>
     </joint>
